Commit message: Got Diff Drive Example working

File: models/krytn/krytn.xacro.urdf (robot description, URDF)
Before this commit: robot krytn, 3 links, 2 joints
Links:
- link base_link: geometry collision box size=0.1 0.07 0.07; collision box size=0.1 0.07 0.07

Commit message: Adjusted URDF so that Realsense Depth Camera works.

File: models/krytn/krytn.xacro.urdf (robot description, URDF)
Before this commit: robot krytn, 3 links, 2 joints
Links:
- added link realsense_depth_link; collision cylinder length=0.05 radius=0.05; visual cylinder length=0.05 radius=0.05
- added link realsense_link
Joints:
- added joint realsense_depth_joint: type fixed, parent realsense_link, child realsense_depth_link, origin xyz=0 0 0 rpy=${-pi/2} 0 ${-pi/2}
- added joint realsense_joint: type fixed, parent base_link, child realsense_link, origin xyz=0 0 0.6 rpy=0 0 0
