Commit message: setting up perception

File: models/krytn/krytn_real.xacro.urdf (robot description, URDF)
Before this commit: robot krytn, 5 links, 4 joints
Links:
- removed link realsense_depth_link
- removed link realsense_link
Joints:
- removed joint realsense_depth_joint
- removed joint realsense_joint
